File: Hardware/DDSFunctionGenerator/DDSFunctionGenerator.kicad_pcb (KiCad board)
At the start: 2 copper layers, 80 x 65 mm, 155 parts, among them J1 Conn_Coaxial, J2 USB_B_Micro, J3 DG128-5.0-02P-14-00A, J4 Conn_01x02_Female, J5 Conn_Coaxial, J6 Conn_Coaxial, J7 Conn_01x04_Male, J8 Conn_01x04_Female, J9 Conn_01x04_Female, Q1 Q_NPN_BEC, Q2 Q_NPN_BEC, Q3 Q_NPN_BEC, SW1 EN11-VSB1AQ15, T1 Transformer_1P_1S, U1 TC1107-3.3VOA, U2 L7805, U3 L78L33_SO8, U4 AD9832, U5 STM32F030K6Tx, U6 FT200XD, U7 AD8325, U8 MCP3425A0T-ECH, X1 XO91, Y1 20MHz

Commit message: pcb ready to be send to fabrication
Parts:
- added H1: MountingHole_Pad, MountingHole:MountingHole_2.5mm_Pad, F.Cu at (105.0, 102.5)
- C24, C25: value 8p -> 8p2
- C56: footprint Capacitor_SMD:C_0603_1608Metric -> Capacitor_SMD:C_0402_1005Metric
- C63, R14: moved to F.Cu
- C64: value 2u2 -> 100n
- R33: footprint Resistor_SMD:R_0805_2012Metric_Pad1.15x1.40mm_HandSolder -> Resistor_SMD:R_0402_1005Metric
- U2: value L7805 -> L78L08_SOT89
- moved C6 6.77 mm to (143.4, 113.4), turned to -90 degrees
- moved U2 0.11 mm to (141.8, 109.9), turned to 90 degrees
Connections:
- C39 pad 1: ROT_B -> ROT_A
- R8 pad 1: ROT_B -> ROT_A
- U2 pad 1: 9V -> 5V_ANALOG
- U2 pad 3: 5V_ANALOG -> 9V
- U5 pad 26: ROT_B -> ROT_A
Routing:
- net ROT_B: track 31.0 -> 0.00 mm
- net ROT_A: track 30.3 -> 61.3 mm
- net 9V: track 106.9 -> 112.2 mm, vias 2 -> 1
- net SPI1_MOSI: track 66.4 -> 70.7 mm
- net SPI1_SCK: track 66.8 -> 70.7 mm
- net SPI1_CS_AMPLIFIER: track 22.8 -> 26.6 mm
- net 5V_ANALOG: track 128.9 -> 132.0 mm
- net 5V_DIGITAL: track 173.1 -> 175.4 mm, vias 2 -> 3
- net SDA: track 67.6 -> 68.1 mm
- net GND: track 61.0 -> 60.7 mm, vias 77 -> 75
Other:
- net class Default removed
- net class rf_power_supply removed
- board text added: "1"
- board text added: "DDS Function Generator rev 1.0"
- board text added: "LCD (Vcc, SCL, SCA, GND)"
- board text added: "PROG (NRST, GND, SWCLK, SWDIO)"
- board text added: "UART(Vcc, TX, RX, GND)"
